Commit message: feat: singularity-safe IK, joint-space homing & regularization
- Custom position-only Jacobian pseudo-inverse IK (damped 3x4) replacing
  KDL LMA for 4-DOF arm; null-space bias keeps arm near seed config
- Backward-walk seeding (end→start) ensures correct elbow-down solution
- Joint-space PD homing mode prevents Cartesian impedance arm flips
- Joint-space regularization during MOVE/WAIT improves z-tracking ~40%
- Gazebo verified: controller active, state machine cycles, EE x>0 always
- Updated .gitignore, README.md, project_status.md

File: ws/src/open_manipulator/open_manipulator_x_description/ros2_control/open_manipulator_x_system.ros2_control.xacro (robot description, xacro)
@@ -1,12 +1,12 @@
 <?xml version="1.0"?>
 <robot xmlns:xacro="http://www.ros.org/wiki/xacro">
-  <xacro:macro name="open_manipulator_x_system" params="name prefix port_name:=/dev/ttyUSB0 use_sim:=^|false use_fake_hardware:=^|false fake_sensor_commands:=^|false">
+  <xacro:macro name="open_manipulator_x_system" params="name prefix port_name:=/dev/ttyUSB0 use_sim:=false use_fake_hardware:=false fake_sensor_commands:=false">
     <ros2_control name="${name}" type="system">
-      <xacro:if value="$(arg use_sim)">
+      <xacro:if value="${use_sim}">
         <hardware>
           <plugin>gazebo_ros2_control/GazeboSystem</plugin>
         </hardware>
       </xacro:if>
-      <xacro:unless value="$(arg use_sim)">
+      <xacro:unless value="${use_sim}">
         <hardware>
           <xacro:if value="${use_fake_hardware}">
@@ -19,5 +19,4 @@
             <param name="port_name">${port_name}</param>
             <param name="baud_rate">1000000</param>
-            <param name="disable_torque_at_init">true</param>
             <param name="error_timeout_sec">0.2</param>
             <param name="dynamixel_model_folder">/param/dxl_model</param>
@@ -58,5 +57,4 @@
       </xacro:unless>
       <joint name="${prefix}joint1">
-        <!-- <command_interface name="position"/> -->
         <command_interface name="effort"/>
         <state_interface name="position"/>
@@ -65,5 +63,4 @@
       </joint>
       <joint name="${prefix}joint2">
-        <!-- <command_interface name="position"/> -->
         <command_interface name="effort"/>
         <state_interface name="position"/>
@@ -72,5 +69,4 @@
       </joint>
       <joint name="${prefix}joint3">
-        <!-- <command_interface name="position"/> -->
         <command_interface name="effort"/>
         <state_interface name="position"/>
@@ -79,5 +75,4 @@
       </joint>
       <joint name="${prefix}joint4">
-        <!-- <command_interface name="position"/> -->
         <command_interface name="effort"/>
         <state_interface name="position"/>
@@ -99,9 +94,8 @@
         <state_interface name="effort"/>
       </joint>
-      <!-- Current Control Mode (Operating Mode = 0) for gravity compensation -->
       <gpio name="dxl1">
         <param name="type">dxl</param>
         <param name="ID">11</param>
-        <command_interface name="Goal Current"/>
+        <command_interface name="Goal Position"/>
         <state_interface name="Present Position"/>
         <state_interface name="Present Velocity"/>
@@ -109,5 +103,9 @@
         <state_interface name="Torque Enable"/>
         <state_interface name="Present Input Voltage"/>
-        <param name="Operating Mode">0</param>
+        <param name="Position P Gain">800</param>
+        <param name="Position I Gain">100</param>
+        <param name="Position D Gain">100</param>
+        <param name="Profile Velocity">200</param>
+        <param name="Profile Acceleration">50</param>
         <param name="Drive Mode">0</param>
         <param name="Return Delay Time">0</param>
@@ -116,5 +114,5 @@
         <param name="type">dxl</param>
         <param name="ID">12</param>
-        <command_interface name="Goal Current"/>
+        <command_interface name="Goal Position"/>
         <state_interface name="Present Position"/>
         <state_interface name="Present Velocity"/>
@@ -122,5 +120,9 @@
         <state_interface name="Torque Enable"/>
         <state_interface name="Present Input Voltage"/>
-        <param name="Operating Mode">0</param>
+        <param name="Position P Gain">800</param>
+        <param name="Position I Gain">100</param>
+        <param name="Position D Gain">100</param>
+        <param name="Profile Velocity">200</param>
+        <param name="Profile Acceleration">50</param>
         <param name="Drive Mode">0</param>
         <param name="Return Delay Time">0</param>
@@ -129,5 +131,5 @@
         <param name="type">dxl</param>
         <param name="ID">13</param>
-        <command_interface name="Goal Current"/>
+        <command_interface name="Goal Position"/>
         <state_interface name="Present Position"/>
         <state_interface name="Present Velocity"/>
@@ -135,5 +137,9 @@
         <state_interface name="Torque Enable"/>
         <state_interface name="Present Input Voltage"/>
-        <param name="Operating Mode">0</param>
+        <param name="Position P Gain">800</param>
+        <param name="Position I Gain">100</param>
+        <param name="Position D Gain">100</param>
+        <param name="Profile Velocity">200</param>
+        <param name="Profile Acceleration">50</param>
         <param name="Drive Mode">0</param>
         <param name="Return Delay Time">0</param>
@@ -142,5 +148,5 @@
         <param name="type">dxl</param>
         <param name="ID">14</param>
-        <command_interface name="Goal Current"/>
+        <command_interface name="Goal Position"/>
         <state_interface name="Present Position"/>
         <state_interface name="Present Velocity"/>
@@ -148,5 +154,9 @@
         <state_interface name="Torque Enable"/>
         <state_interface name="Present Input Voltage"/>
-        <param name="Operating Mode">0</param>
+        <param name="Position P Gain">800</param>
+        <param name="Position I Gain">100</param>
+        <param name="Position D Gain">100</param>
+        <param name="Profile Velocity">200</param>
+        <param name="Profile Acceleration">50</param>
         <param name="Drive Mode">0</param>
         <param name="Return Delay Time">0</param>

File: ws/src/open_manipulator/open_manipulator_x_description/urdf/open_manipulator_x_robot.urdf.xacro (robot description, xacro)
@@ -1,5 +1,8 @@
 <?xml version="1.0"?>
-<!-- OpenManipulator Chain -->
+<!-- OpenManipulator-X Unified Robot Description -->
 <robot name="open_manipulator_x" xmlns:xacro="http://ros.org/wiki/xacro">
+  <!-- ======================== -->
+  <!-- Arguments -->
+  <!-- ======================== -->
   <xacro:arg name="prefix" default="" />
   <xacro:arg name="use_sim" default="false" />
@@ -7,34 +10,56 @@
   <xacro:arg name="fake_sensor_commands" default="false" />
   <xacro:arg name="port_name" default="/dev/ttyUSB0" />
-  <xacro:arg name="controller_config" default="$(find open_manipulator_x_bringup)/config/gazebo_controller_manager.yaml" />
-  <xacro:arg name="robot_namespace" default="" />
-  <!-- Import Rviz colors -->
+  <xacro:arg name="controller_config"
+             default="$(find open_manipulator_x_bringup)/config/gazebo_controller_manager.yaml" />
+  <!-- ======================== -->
+  <!-- Includes -->
+  <!-- ======================== -->
+  <!-- Gazebo materials -->
   <xacro:include filename="$(find open_manipulator_x_description)/gazebo/materials.xacro" />
-  <!-- Import all Gazebo-customization elements, including Gazebo colors -->
+  <!-- Gazebo visual + physics customizations -->
   <xacro:include filename="$(find open_manipulator_x_description)/gazebo/open_manipulator_x.gazebo.xacro" />
-  <!-- Import URDF -->
+  <!-- Core URDF -->
   <xacro:include filename="$(find open_manipulator_x_description)/urdf/open_manipulator_x.urdf.xacro" />
+  <!-- ros2_control system -->
   <xacro:include filename="$(find open_manipulator_x_description)/ros2_control/open_manipulator_x_system.ros2_control.xacro" />
+  <!-- ======================== -->
+  <!-- Robot Model -->
+  <!-- ======================== -->
   <xacro:open_manipulator_x prefix="$(arg prefix)" />
+  <!-- Gazebo-specific elements (collision tweaks, friction, etc.) -->
   <xacro:open_manipulator_x_gazebo prefix="$(arg prefix)" />
+  <!-- ros2_control hardware interface -->
   <xacro:open_manipulator_x_system
-    name="OpenManipulatorXSystem_$(arg robot_namespace)" prefix="$(arg prefix)" use_sim="$(arg use_sim)"
+    name="OpenManipulatorXSystem"
+    prefix="$(arg prefix)"
+    use_sim="$(arg use_sim)"
     use_fake_hardware="$(arg use_fake_hardware)"
     fake_sensor_commands="$(arg fake_sensor_commands)"
-    port_name="$(arg port_name)"/>
+    port_name="$(arg port_name)"
+  />
+  <!-- ======================== -->
+  <!-- Gazebo ros2_control Plugin -->
+  <!-- ======================== -->
+  <!--
+    IMPORTANT:
+    - This MUST be present when use_sim:=true.
+    - Do NOT launch standalone ros2_control_node in simulation.
+    - Gazebo will create controller_manager internally.
+  -->
+  <xacro:if value="$(arg use_sim)">
   <gazebo>
-  <plugin name="gazebo_ros2_control_$(arg robot_namespace)" filename="libgazebo_ros2_control.so">
-    <parameters>$(arg controller_config)</parameters>
-      <robot_param>robot_description</robot_param>
-      <robot_param_node>/$(arg robot_namespace)/robot_state_publisher</robot_param_node>
-    <robot_namespace>/$(arg robot_namespace)</robot_namespace>
-    <ros>
-      <namespace>/$(arg robot_namespace)</namespace>
-    </ros>
-  </plugin>
-</gazebo>
-  <!-- World -->
+    <plugin name="gazebo_ros2_control"
+            filename="libgazebo_ros2_control.so">
+      <ros>
+        <namespace>/omx</namespace>
+      </ros>
+      <parameters>$(arg controller_config)</parameters>
+    </plugin>
+  </gazebo>
+  </xacro:if>
+  <!-- ======================== -->
+  <!-- World Attachment -->
+  <!-- ======================== -->
   <link name="world"/>
-  <!-- World fixed joint-->
   <joint name="$(arg prefix)world_fixed" type="fixed">
     <origin xyz="0 0 0" rpy="0 0 0"/>
